File: boards/spectrometer/spectrometer.kicad_sch (KiCad schematic)
At the start: 0 parts

Commit message: references
Parts:
- added B1: KMR2, Button_Switch_SMD:SW_Push_1P1T_NO_CK_KMR2, symbol Switch:SW_Push
- added BT1: 3V, BITSv5:SEIKO_ML414H_IV01E, symbol Device:Battery_Cell
- added C1, C11, C13, C14, C15, C16, C18, C20, C4, C7, C9: 100nF, Capacitor_SMD:C_0402_1005Metric, symbol Device:C_Small
- added C2, C3: 10pF, Capacitor_SMD:C_0402_1005Metric, symbol Device:C_Small
- added C25, C29: 100nF, Capacitor_SMD:C_0603_1608Metric, symbol Device:C_Small
- added C33, C35, C8: 1uF, Capacitor_SMD:C_0603_1608Metric, symbol Device:C_Small
- added C5, C6: 1uF, Capacitor_SMD:C_0402_1005Metric, symbol Device:C_Small
- added D1: LED, LED_SMD:LED_0603_1608Metric, symbol Device:LED
- added D2: 0.5A/40V/240mV, Diode_SMD:D_SOD-123F, symbol Device:D_Schottky_Small
- added H1, H2: M2, MountingHole:MountingHole_2.2mm_M2_Pad, symbol Mechanical:MountingHole
- added H3: M2, MountingHole:MountingHole_2.2mm_M2_Pad, symbol Mechanical:MountingHole_Pad
- added J1: USB_C_Receptacle_USB2.0, Connector_USB:USB_C_Receptacle_GCT_USB4105-xx-A_16P_TopMnt_Horizontal, symbol Connector:USB_C_Receptacle_USB2.0
- added J2: XT30, Connector_AMASS:AMASS_XT30PW-M_1x02_P2.50mm_Horizontal, symbol Connector_Generic:Conn_01x02
- added J3: Conn_01x02, symbol Connector_Generic:Conn_01x02
- added J6: U.FL, Connector_Coaxial:U.FL_Molex_MCRF_73412-0110_Vertical, symbol Connector:Conn_Coaxial
- added Q1: Q_NMOS_GSD, Package_TO_SOT_SMD:SOT-23-3, symbol Device:Q_NMOS_GSD
- added R1: 1K, Resistor_SMD:R_0402_1005Metric, symbol Device:R_Small
- added R10: 44.2K, Resistor_SMD:R_0603_1608Metric, symbol Device:R_Small
- added R11, R14, R15, R16, R17, R18, R7, R8: idk, symbol Device:R_Small
- added R12: 1K, Resistor_SMD:R_0603_1608Metric, symbol Device:R_Small
- added R13, R23, R24: DNF, Resistor_SMD:R_0603_1608Metric, symbol Device:R_Small
- added R2: 10k, Resistor_SMD:R_0603_1608Metric, symbol Device:R_Small
- added R3, R4: 5.1K, Resistor_SMD:R_0603_1608Metric_Pad0.98x0.95mm_HandSolder, symbol Device:R_Small
- added R30: 3.3K, Resistor_SMD:R_0603_1608Metric, symbol Device:R_Small
- added R5, R6: 27, Resistor_SMD:R_0402_1005Metric, symbol Device:R_Small
- added R9: 470, Resistor_SMD:R_0603_1608Metric, symbol Device:R_Small
- added SW2: ~, BITSv5:CAS-120TB_NDC-M, symbol Switch:SW_SPDT
- added TP1, TP2, TP5: TestPoint, TestPoint:TestPoint_Keystone_5000-5004_Miniature, symbol Connector:TestPoint
- added TP3, TP4: TestPoint, TestPoint:TestPoint_Pad_D2.0mm, symbol Connector:TestPoint
- added U1: C12880MA, symbol BPP_Lib:C12880MA
- added U10: MS5607-02BA, Package_LGA:LGA-8_3x5mm_P1.25mm, symbol Sensor_Pressure:MS5607-02BA
- added U12: MAX-M10S, RF_GPS:ublox_MAX, symbol RF_GPS:MAX-M10S
- added U2: MCU_RaspberryPi_RP2040_RP2040, BITSv5:RP2040-QFN-56, symbol BITSv5:MCU_RaspberryPi_RP2040
- added U3: TPS2121RUXR, BITSv5:TPS2121, symbol BPP_Lib:TPS2121RUXR
- added U4: USBLC6-2SC6, SOT23-6L_STM, symbol BPP_Lib:USBLC6-2SC6
- added U5: ADS8681IRUMR, RUM0016B, symbol BPP_Lib:ADS8681IRUMR
- added U6: W25Q128JVS, BITSv5:WSON_128JVPIQ_WIN, symbol Memory_Flash:W25Q128JVS
- added U7: LT8653SIV-PBF, 05-08-1524_ADI, symbol BPP_Lib:LT8653SIV-PBF
- added U8: MB85RS1MT, BPP_Lib:BGA8CP30X40_5X3_309X228X35B25N, symbol Memory_NVRAM:MB85RS1MT
- added Y1: 12MHz, Crystal:Crystal_SMD_2520-4Pin_2.5x2.0mm, symbol Device:Crystal_GND24_Small
Connections:
- new net: C8.1, U3.11 (SS)
- new net: D1.2 (A), R9.2
- new net: R11.2, R16.1, U3.4 (OV2)
- new net: J1.A7 (D-), J1.B7 (D-), U4.4 (DI-)
- new net: J1.A6 (D+), J1.B6 (D+), U4.6 (DI+)
- new net: J6.1 (In), U12.11 (RF_IN)
- new net: R17.2, R18.1, U3.3 (CP2)
- new net: C3.1, R1.1, Y1.1
- new net: R12.1, SW2.2 (B)
- new net: C2.1, U2.20 (XIN), Y1.3
- new net: R14.1, R15.2, U3.5 (OV1)
- new net: BT1.1 (+), C35.1, R30.2, U12.6 (V_BCKP)
- new net: B1.2, R2.2, U2.26 (RUN)
- new net: J1.A5 (CC1), R3.2
- new net: D1.1 (K), Q1.3 (D)
- new net: R10.1, U3.10 (ILM)
- new net: U12.10 (GND), U12.12 (GND)
- new net: J1.B5 (CC2), R4.1
- new net: D2.1 (K), R30.1
- new net: R6.2, U2.46 (USB_DM)
- new net: R7.2, R8.1, U3.6 (PR1)
- new net: R5.2, U2.47 (USB_DP)
- new net: R1.2, U2.21 (XOUT)
- new net +1V1: C1.1, C4.1, C5.1, U2.23 (DVDD), U2.45 (VREG_VOUT), U2.50 (DVDD)
- new net +3V3: C11.1, C13.1, C14.1, C15.1, C16.1, C18.1, C20.1, C25.1, C29.1, C33.1, C6.1, C7.1, C9.1, D2.2 (A), R13.2, R2.1, R23.1, R24.1, R9.1, TP2.1, U10.1 (VDD), U10.2 (PS), U12.7 (VCC_IO), U12.8 (VCC), U2.1 (IOVDD), U2.10 (IOVDD), U2.22 (IOVDD), U2.33 (IOVDD), U2.42 (IOVDD), U2.43 (ADC_AVDD), U2.44 (VREG_IN), U2.48 (USB_VDD), U2.49 (IOVDD), U6.8 (VCC), U8.E3 (VDD)
- new net +5V: TP1.1
- new net +BATT: J2.2 (Pin_2), R11.1, R17.1, U3.2 (IN2)
- new net BATT_REG: TP5.1
- new net DRF_BUSY: U2.14 (GPIO11)
- new net DRF_CS: U2.37 (GPIO25)
- new net DRF_DIO1: U2.13 (GPIO10)
- new net DRF_SW: U2.12 (GPIO9)
- new net DRF_TXEN: U2.11 (GPIO8)
- new net EXTINT: U12.5 (EXTINT), U2.29 (GPIO18)
- new net FRAM_CS: U2.41 (GPIO29_ADC3), U8.E1 (~{CS})
- new net GND: B1.1, BT1.2 (-), C1.2, C11.2, C13.2, C14.2, C15.2, C16.2, C18.2, C2.2, C20.2, C25.2, C29.2, C3.2, C33.2, C35.2, C4.2, C5.2, C6.2, C7.2, C8.2, C9.2, H3.1, J1.A1 (GND), J1.A12 (GND), J1.B1 (GND), J1.B12 (GND), J1.S1 (SHIELD), J2.1 (Pin_1), J6.2 (Ext), Q1.2 (S), R10.2, R14.2, R16.2, R18.2, R3.1, R4.2, R8.2, SW2.3 (C), U10.3 (GND), U10.4 (CSB), U10.5 (CSB), U12.1 (GND), U12.10 (GND), U12.12 (GND), U2.19 (TESTEN), U2.57 (GND), U3.12 (GND), U3.9 (ST), U4.2 (GND), U6.4 (GND), U8.A1 (GND), Y1.2, Y1.4
- new net IRIDIUM_CTS: U2.4 (GPIO2)
- new net IRIDIUM_NETAV: U2.6 (GPIO4)
- new net IRIDIUM_RING: U2.7 (GPIO5)
- new net IRIDIUM_RTS: U2.5 (GPIO3)
- new net IRIDIUM_RXD: U2.3 (GPIO1)
- new net IRIDIUM_TXD: U2.15 (GPIO12)
- new net LED: Q1.1 (G), U2.2 (GPIO0)
- new net MISO: U2.36 (GPIO24), U8.C1 (SO)
- new net MOSI: U2.39 (GPIO27_ADC1), U8.A3 (SI)
- new net QSPI_SCLK: U2.52 (QSPI_SCLK), U6.6 (CLK)
- new net QSPI_SD0: U2.53 (QSPI_SD0), U6.5 (DI(IO0))
- new net QSPI_SD1: U2.55 (QSPI_SD1), U6.2 (DO(IO1))
- new net QSPI_SD2: U2.54 (QSPI_SD2), U6.3 (IO2)
- new net QSPI_SD3: U2.51 (QSPI_SD3), U6.7 (IO3)
- new net QSPI_SS: R12.2, R13.1, U2.56 (QSPI_SS), U6.1 (~{CS})
- new net RDIO_RST: U2.16 (GPIO13)
- new net RP_SWCLK: TP3.1, U2.24 (SWCLK)
- new net RP_SWD: TP4.1, U2.25 (SWD)
- new net SCK: U2.38 (GPIO26_ADC0), U8.C3 (SCK)
- new net SCL: R23.2, U10.8 (SCLK), U2.32 (GPIO21)
- new net SDA: R24.2, U10.7 (SDI/SDA), U2.31 (GPIO20)
- new net TIMEPULSE: U12.4 (TIMEPULSE), U2.28 (GPIO17)
- new net USB_D+: R5.1, U4.1 (DO+)
- new net USB_D-: R6.1, U4.3 (DO-)
- new net VBUS: J1.A4 (VBUS), J1.A9 (VBUS), J1.B4 (VBUS), J1.B9 (VBUS), R15.1, R7.1, U3.7 (IN1), U4.5 (Vs)
- no-connect marks 0 -> 22
Other:
- note added: "MCU"

Commit message: more refernces and board stuff
Parts:
- added C10, C17, C19, C21: 4.7pF, symbol Device:C_Small
- added C12, C22: 470pF, symbol Device:C_Small
- added C23, C27, C30, C32: 1uF, symbol Device:C_Small
- added C24: 22nF, symbol Device:C_Small
- added C26, C28, C31: 10uF, symbol Device:C_Small
- added C34: C_Small, symbol Device:C_Small
- added C36, C37: 100nF, symbol Device:C_Small
- added L1, L2: 2.2uH, symbol Device:L_Small
- added L3, L4: 3.3uH, symbol Device:L_Small
- added R19, R20: 34.8k, symbol Device:R_Small
- added R21, R27: 1M, symbol Device:R_Small
- added R22: 191k, symbol Device:R_Small
- added R25, R26: 100k, symbol Device:R_Small
- added R28: 316k, symbol Device:R_Small
- added R29: 15k, symbol Device:R_Small
- added R31, R32: 100m, symbol Device:R_Small
- added R33, R34: idk, Resistor_SMD:R_0603_1608Metric, symbol Device:R_Small
- added R35: 100k, Resistor_SMD:R_0603_1608Metric, symbol Device:R_Small
- U2: value MCU_RaspberryPi_RP2040_RP2040 -> MCU_RaspberryPi_RP2040; symbol BITSv5:MCU_RaspberryPi_RP2040 -> BPP_Lib:MCU_RaspberryPi_RP2040
- U5: value ADS8681IRUMR -> ADS8681
- U7: value LT8653SIV-PBF -> LT8653SIV
Connections:
- net +5V: now also C30.1, L3.2, R31.2
- net +BATT: now also R33.2
- net GND: now also U5.1 (AGND), U5.15 (DGND), U5.17 (PAD), U7.1 (D0), U7.2 (D1), U7.21 (GND), C10.2, C12.2, C17.2, C22.2, C23.2, C24.2, C26.2, C27.2, C28.2, C30.2, C31.2, C32.2, R22.2, R28.2, R29.2, R34.1
- net VBUS: now also R35.2
- net at U5.2 (REFIO): now also C37.1
- net at U5.3 (REFGND): now also C36.2, C37.2
- net at U5.4 (REFCAP): now also C36.1
- net at U5.5 (AIN_P): now also C34.1
- net at U5.6 (AIN_GND): now also C34.2
- net at U7.11 (VC1): now also C10.1, R19.1
- net at U7.12 (FB1): now also C21.2, R21.2, R22.1
- net at U7.13 (SS1): now also U7.14 (SS2), C24.1
- net at U7.15 (FB2): now also C19.2, R27.2, R28.1
- net at U7.16 (VC2): now also C17.1, R20.1
- net at U7.17 (RT): now also R29.1
- net at U7.18 (EN/UV): now also R33.1, R34.2, R35.1
- net at U7.19 (VIN): now also U3.1 (OUT), U3.8 (OUT), U7.20 (VIN), C26.1, C27.1
- net at U7.3 (PG2): now also R26.1
- net at U7.4 (PG1): now also R25.1
- net at U7.7 (SW1): now also L1.1
- net at U7.8 (SW2): now also L2.1
- net at U7.9 (VCC): now also C23.1
- new net: C12.1, R19.2
- new net: C22.1, R20.2
- new net: C21.1, C28.1, L1.2, L3.1, R21.1, R25.2, R31.1
- new net: C19.1, C31.1, L2.2, L4.1, R26.2, R27.1, R32.1
- new net: U12.10 (GND), U12.12 (GND)
- new net +3.3V: C32.1, L4.2, R32.2
- no-connect marks 22 -> 24
Other:
- note added: "8 x 100nF"
- note removed: "MCU"
- moved on the sheet: B1, R2
